Commit message: ..

File: description/robot_core.xacro (robot description, xacro)
@@ -6,5 +6,5 @@
     <xacro:property name="chassis_height" value="0.065"/>
     <xacro:property name="chassis_mass" value="1.0"/>
-    <xacro:property name="wheel_radius" value="0.033"/>
+    <xacro:property name="wheel_radius" value="0.034"/>
     <xacro:property name="wheel_thickness" value="0.021"/>
     <xacro:property name="wheel_mass" value="0.05"/>

File: description/ros2_control.xacro (robot description, xacro)
@@ -11,5 +11,5 @@
                 <param name="baud_rate">57600</param>
                 <param name="timeout">1000</param>
-                <param name="enc_counts_per_rev">3436</param>
+                <param name="enc_counts_per_rev">3440</param>
             </hardware>
             <joint name="left_wheel_joint">

Commit message: s

File: description/robot_core.xacro (robot description, xacro)
@@ -10,5 +10,5 @@
     <xacro:property name="wheel_mass" value="0.05"/>
     <xacro:property name="wheel_offset_x" value="0.171"/>
-    <xacro:property name="wheel_offset_y" value="0.115"/>
+    <xacro:property name="wheel_offset_y" value="0.1125"/>
     <!-- <xacro:property name="wheel_offset_z" value="0.027"/> -->
     <!-- <xacro:property name="chassis_bottom_z" value="0.025"/> -->
