Commit message: Add base_footprint link and slam_toolbox params; save RViz layout
- robot_core.xacro: base_footprint (fixed, zero offset under base_link), as in
  the articubot_one reference; needed by slam_toolbox/AMCL base_frame.
- config/mapper_params_mapping.yaml: stock Foxy slam_toolbox params, mode
  mapping, max_laser_range 12 for the YDLIDAR X2 (use for building new maps).
- config/mapper_params_online_async.yaml: localization-mode variant pointing at
  the serialized sim map.
- config/main.rviz: saved layout with the Map display.

Co-Authored-By: Claude Sonnet 5.5 <noreply@anthropic.com>

File: description/robot_core.xacro (robot description, xacro)
@@ -36,4 +36,12 @@
     <!-- BASE LINK -->
     <link name="base_link">
+    </link>
+    <!-- BASE_FOOTPRINT LINK -->
+    <joint name="base_footprint_joint" type="fixed">
+        <parent link="base_link"/>
+        <child link="base_footprint"/>
+        <origin xyz="0 0 0" rpy="0 0 0"/>
+    </joint>
+    <link name="base_footprint">
     </link>
     <!-- CHASSIS LINK -->
