Commit message: Robot model and sizes for the new delivery body
Measured 2026-10-23: box 0.33 x 0.244 x 0.19 m (board 0.046 above the floor), drive
wheels at the front (axle 0.085 from the front edge), tyre centres 0.288 apart,
21 mm swivel caster 0.165 behind the axle, lidar centred on top of the box 0.1995
behind the axle (beam about 0.272 above the floor).

- robot_core/lidar/camera xacro: new dimensions (old values kept in comments; no
  colon-space in comments, Foxy parses robot_description as YAML first)
- my_controllers: wheel_separation 0.225 -> 0.288, multiplier 1.055 -> 1.0 (to be
  recalibrated with a 360 degree turn); wheel_radius stays 0.034 (1 m tape test)
- nav2: robot_radius 0.22 -> 0.29 (the back corner sweeps 0.274 around the axle)
- drive/turn test tools: same wheel numbers

Checked: xacro + check_urdf, part positions against the measurements, rsp launch and
RViz with joint_state_publisher_gui.

Co-Authored-By: Claude Opus 5.5 <noreply@anthropic.com>

File: description/camera.xacro (robot description, xacro)
@@ -4,5 +4,5 @@
         <parent link="chassis"/>
         <child link="camera_link"/>
-        <origin xyz="0.305 0 0.08" rpy="0 0 0"/>
+        <origin xyz="0.33 0 0.08" rpy="0 0 0"/>   <!-- simulation only, front face of the box (old robot 0.305) -->
     </joint>
     <link name="camera_link">

File: description/lidar.xacro (robot description, xacro)
@@ -4,6 +4,8 @@
         <parent link="chassis"/>
         <child link="laser_frame"/>
-        <origin xyz="0.058 0 0.103" rpy="0 0 0"/>
-        <!-- <origin xyz="0.058 0 0.103" rpy="0 0 0"/>  -->
+        <!-- on top of the delivery box, centred, 0.0455 from the back edge (0.1995 behind the axle);
+             beam about 0.272 above the floor = 0.226 above the board bottom (box top 0.236, cap top 0.2855) -->
+        <origin xyz="0.0455 0 0.226" rpy="0 0 0"/>
+        <!-- old robot had xyz 0.058 0 0.103 (no colons in comments - Foxy reads the model as YAML first) -->
     </joint>
     <link name="laser_frame">

File: description/robot_core.xacro (robot description, xacro)
@@ -2,19 +2,23 @@
 <robot xmlns:xacro="http://www.ros.org/wiki/xacro" >
     <xacro:include filename="inertial_macros.xacro"/>
-    <xacro:property name="chassis_length" value="0.273"/>
-    <xacro:property name="chassis_width" value="0.203"/>
-    <xacro:property name="chassis_height" value="0.065"/>
+    <!-- Delivery body, measured 2026-10-23. base_link = middle of the drive axle (drive wheels at the FRONT).
+         Old robot (before 2026-10-23) had length 0.273, width 0.203, height 0.065, wheel_offset_x 0.171,
+         wheel_offset_y 0.1125, chassis_bottom_z = wheel_radius, caster 0.011 at x 0.030.
+         Never write a colon followed by a space in these files - Foxy reads the model as YAML first and fails. -->
+    <xacro:property name="chassis_length" value="0.33"/>     <!-- front edge to back edge -->
+    <xacro:property name="chassis_width" value="0.244"/>     <!-- without the wheels -->
+    <xacro:property name="chassis_height" value="0.19"/>     <!-- board bottom 0.046 to box top 0.236 above the floor -->
     <xacro:property name="chassis_mass" value="1.0"/>
-    <xacro:property name="wheel_radius" value="0.034"/>
-    <xacro:property name="wheel_thickness" value="0.021"/>
+    <xacro:property name="wheel_radius" value="0.034"/>      <!-- 70 mm wheels; 0.034 matched a 1 m tape test under load -->
+    <xacro:property name="wheel_thickness" value="0.023"/>
     <xacro:property name="wheel_mass" value="0.05"/>
-    <xacro:property name="wheel_offset_x" value="0.171"/>
-    <xacro:property name="wheel_offset_y" value="0.1125"/>
+    <xacro:property name="wheel_offset_x" value="0.245"/>    <!-- axle to the BACK edge (axle is 0.085 from the front) -->
+    <xacro:property name="wheel_offset_y" value="0.144"/>    <!-- half of 0.288, tyre centre to tyre centre -->
     <!-- <xacro:property name="wheel_offset_z" value="0.027"/> -->
     <!-- <xacro:property name="chassis_bottom_z" value="0.025"/> -->
-    <xacro:property name="chassis_bottom_z" value="${wheel_radius}"/>
-    <xacro:property name="caster_wheel_radius" value="0.011"/>
+    <xacro:property name="chassis_bottom_z" value="0.011"/>  <!-- board bottom above the axle: 0.046 floor-to-board minus 0.035 -->
+    <xacro:property name="caster_wheel_radius" value="0.0105"/>  <!-- 21 mm swivel caster -->
     <xacro:property name="caster_wheel_mass" value="0.01"/>
-    <xacro:property name="caster_wheel_offset_x" value="0.030"/>
+    <xacro:property name="caster_wheel_offset_x" value="0.080"/> <!-- from the back edge: 0.165 behind the axle -->
     <!-- <xacro:property name="caster_wheel_offset_z" value="${wheel_offset_z - wheel_radius + caster_wheel_radius}"/> -->
     <xacro:property name="caster_wheel_offset_z" value="${-wheel_radius + caster_wheel_radius - chassis_bottom_z}"/>
